File: kicad source files/pico-modxo.kicad_sch (KiCad schematic)
At the start: 14 parts, among them J1 XBOX_LPC, U1 RP2040-Zero

Commit message: Added traces for V1.0
Added traces for V1.0
Parts:
- removed D0: D0, Connector_Wire:SolderWirePad_1x01_SMD_1x2mm, symbol Connector:Conn_01x01_Pin
- removed D1: D_Schottky, Diode_THT:D_DO-41_SOD81_P7.62mm_Horizontal, symbol Device:D_Schottky
- removed D2: LED, LED_THT:LED_D4.0mm, symbol Device:LED
- removed JP1, JP2, JP3: ~, Jumper:SolderJumper-2_P1.3mm_Open_RoundedPad1.0x1.5mm, symbol Jumper:SolderJumper_2_Open
- removed LFrame1: ~, Connector_Wire:SolderWirePad_1x01_SMD_1x2mm, symbol Connector:Conn_01x01_Pin
- removed R5: 1kΩ, Resistor_THT:R_Axial_DIN0204_L3.6mm_D1.6mm_P7.62mm_Horizontal, symbol Device:R
- added D0: D0 (V1.0-V1.5), TestPoint:TestPoint_Pad_4.0x4.0mm, symbol Connector:Conn_01x01_Female
- added D1: RB551VM-30TE-17, Diode_SMD:D_MELF-RM10_Universal_Handsoldering, symbol Device:D
- J1: footprint xbox_lpc:XBOX_LPC -> xbox_lpc:xbox_lpc
- R1, R2, R3, R4: footprint Resistor_THT:R_Axial_DIN0204_L3.6mm_D1.6mm_P7.62mm_Horizontal -> Resistors_Universal:Resistor_SMD+THTuniversal_1206_RM10_HandSoldering
- U1: value RP2040-Zero -> rp2040-zero
Connections:
- net +5V: now also D1.1 (K)
- net GND: now also J1.12 (GND)
- net at J1.6 (5V): now also D1.2 (A)
- net at U1.7 (6): now also D0.1 (Pin_1)
- net LRESET: now reaches U1.8 (7)
- net LRESET: now also J1.5 (LRESET#)
- net +3.3V: now reaches U1.9 (8)
- net +3.3V: now also J1.15 (3.3V), J1.9 (3.3V)
- net LSDA: now reaches J1.14 (SDA)
- net LSCL: now reaches J1.13 (SCL)
- net SCL1: no longer names the net of U1.18 (27)
- net SDA1: no longer names the net of U1.17 (26)
- no-connect marks 17 -> 2
Other:
- note added: "RP2040-Zero"
- note removed: "(V1.0 - V1.5 only)"
- note removed: "Special thanks to: ShalX modzvilleusa consolemods.org r/XboxModding Xbox modding scene Rocky5"
- note removed: "https://consolemods.org/wiki/Xbox:ModXo https://github.com/shalxmva/modxo https://github.com/Electrical5/ModXo-RP2040-Zero"
- company: OpenSource (GNU GPL3.0) -> Simplified version (no RGB/LED/display/io)
- title: ModXo RP2040-Zero -> Pi Pico adapter for ModXo
