File: Kicad Source Files/modxo-rp2040.kicad_sch (KiCad schematic)
At the start: 8 parts, among them J1 XBOX_LPC, U1 rp2040-zero

Commit message: Added logos
Parts:
- D0: value D0 (V1.0-V1.5) -> (V1.0-V1.5); footprint TestPoint:TestPoint_Pad_4.0x4.0mm -> TestPoint:TestPoint_Pad_2.0x2.0mm; symbol Connector:Conn_01x01_Female -> Connector_Generic:Conn_01x01
Connections:
- net LSCL: no longer names the net of J1.13 (SCL)
- net LSDA: no longer names the net of J1.14 (SDA)
- no-connect marks 2 -> 16
Changed lines of the file:
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@@
+	)
+	(no_connect
+		(at 123.19 66.04)
+	)
+	(no_connect
+		(at 123.19 68.58)
 	)
 	(no_connect
@@
 	)
 	(no_connect
+		(at 130.81 73.66)
+	)
+	(no_connect
+		(at 123.19 60.96)
+	)
+	(no_connect
+		(at 140.97 73.66)
+	)
+	(no_connect
+		(at 48.26 53.34)
+	)
+	(no_connect
 		(at 48.26 66.04)
 	)
+	(no_connect
+		(at 123.19 55.88)
+	)
+	(no_connect
+		(at 135.89 73.66)
+	)
+	(no_connect
+		(at 138.43 73.66)
+	)
+	(no_connect
+		(at 60.96 53.34)
+	)
+	(no_connect
+		(at 123.19 53.34)
+	)
+	(no_connect
+		(at 123.19 63.5)
+	)
+	(no_connect
+		(at 133.35 73.66)
+	)
+	(no_connect
+		(at 123.19 58.42)
+	)
 	(wire
 		(pts
@@
 	(wire
 		(pts
-			(xy 45.72 53.34) (xy 48.26 53.34)
-		)
-		(stroke
-			(width 0)
-			(type default)
-		)
-	)
-	(wire
-		(pts
 			(xy 60.96 58.42) (xy 76.2 58.42)
 		)
@@
 		(pts
 			(xy 60.96 50.8) (xy 76.2 50.8)
-		)
-		(stroke
-			(width 0)
-			(type default)
-		)
-	)
-	(wire
-		(pts
-			(xy 60.96 53.34) (xy 63.5 53.34)
 		)
 		(stroke
@@
 		(property "Intersheetrefs" "${INTERSHEET_REFS}"
 			(at 38.1386 60.96 0)
-			(effects
-				(font
-					(size 1.27 1.27)
-				)
-				(justify right)
-				(hide yes)
-			)
-		)
-	)
-	(global_label "LSCL"
-		(shape input)
-		(at 63.5 53.34 0)
-		(fields_autoplaced yes)
-		(effects
-			(font
-				(size 1.27 1.27)
-			)
-			(justify left)
-		)
-		(property "Intersheetrefs" "${INTERSHEET_REFS}"
-			(at 71.0209 53.34 0)
-			(effects
-				(font
-					(size 1.27 1.27)
-				)
-				(justify left)
-				(hide yes)
-			)
-		)
-	)
-	(global_label "LSDA"
-		(shape input)
-		(at 45.72 53.34 180)
-		(fields_autoplaced yes)
-		(effects
-			(font
-				(size 1.27 1.27)
-			)
-			(justify right)
-		)
-		(property "Intersheetrefs" "${INTERSHEET_REFS}"
-			(at 38.1386 53.34 0)
 			(effects
 				(font
@@
 					(size 1.27 1.27)
 				)
-				(hide yes)
 			)
 		)
@@
 	)
 	(symbol
-		(lib_id "Connector:Conn_01x01_Female")
+		(lib_id "Connector_Generic:Conn_01x01")
 		(at 157.48 63.5 0)
 		(unit 1)
@@
 		(dnp no)
 		(property "Reference" "D0"
-			(at 170.688 63.5 0)
-			(effects
-				(font
-					(size 1.27 1.27)
-				)
-				(justify left)
-				(hide yes)
-			)
-		)
-		(property "Value" "D0 (V1.0-V1.5)"
-			(at 158.242 63.5 0)
-			(effects
-				(font
-					(size 1.27 1.27)
-				)
-				(justify left)
-			)
-		)
-		(property "Footprint" "TestPoint:TestPoint_Pad_4.0x4.0mm"
+			(at 160.02 63.5 0)
+			(effects
+				(font
+					(size 1.27 1.27)
+				)
+			)
+		)
+		(property "Value" "(V1.0-V1.5)"
+			(at 167.64 63.5 0)
+			(effects
+				(font
+					(size 1.27 1.27)
+				)
+			)
+		)
+		(property "Footprint" "TestPoint:TestPoint_Pad_2.0x2.0mm"
 			(at 157.48 63.5 0)
 			(effects
@@
 	)
 	(symbol
+		(lib_name "+5V_1")
 		(lib_id "power:+5V")
 		(at 29.21 50.8 0)
@@
 		)
 		(property "Value" "RB551VM-30TE-17"
-			(at 31.75 65.532 0)
+			(at 34.29 65.532 0)
 			(effects
 				(font
@@
 	)
 	(symbol
+		(lib_name "+3.3V_1")
 		(lib_id "power:+3.3V")
 		(at 76.2 50.8 0)
